File: XNP_1/XNP_1.kicad_sch (KiCad schematic)
At the start: 11 parts, among them J2 RJ12, J4 RJ12, J5 RJ12

Commit message: Rozložení na DPS
Parts:
- added H1, H2: MountingHole, MountingHole:MountingHole_3mm_Pad_TopBottom, symbol Mechanical:MountingHole
- C1: value (none) -> 100n; footprint (none) -> Capacitor_SMD:C_0805_2012Metric
- D1: value (none) -> LED; footprint (none) -> LED_THT:LED_D3.0mm_Clear
- J1: value (none) -> RJ12; footprint (none) -> Connector_RJ:RJ12_Amphenol_54601
- J2, J4, J5: footprint (none) -> Connector_RJ:RJ12_Amphenol_54601
- J3: value (none) -> Conn_01x02; footprint (none) -> Connector_PinSocket_2.54mm:PinSocket_1x02_P2.54mm_Vertical
- JP1: value (none) -> SolderJumper_2_Bridged; footprint (none) -> Jumper:SolderJumper-2_P1.3mm_Bridged_RoundedPad1.0x1.5mm
- JP2: value (none) -> SolderJumper_2_Open; footprint (none) -> Jumper:SolderJumper-2_P1.3mm_Open_RoundedPad1.0x1.5mm
- R1: value (none) -> 4k7; footprint (none) -> Resistor_SMD:R_0805_2012Metric
- R2: footprint (none) -> Resistor_SMD:R_0805_2012Metric
Connections:
- no-connect marks 0 -> 8
