File: XNP_1/XNP_1.kicad_pcb (KiCad board)
At the start: 2 copper layers, 57 x 31 mm, 13 parts, among them J1 RJ12, J2 RJ12, J3 Conn_01x02, J4 RJ12, J5 RJ12

Commit message: Dokončen návrh DPS
Parts:
- moved J3 10.8 mm to (124.5, 74.6)
Routing:
- net Net-(C1-Pad2): track 0.00 -> 79.9 mm, vias 0 -> 2
- net Net-(D1-A): track 0.00 -> 74.1 mm, vias 0 -> 3
- net Net-(J3-Pin_1): track 0.00 -> 70.1 mm, vias 0 -> 3
- net Net-(J3-Pin_2): track 0.00 -> 69.6 mm, vias 0 -> 1
- net Net-(D1-K): track 0.00 -> 4.69 mm
- net Net-(JP1-A): track 0.00 -> 3.88 mm
- net Net-(JP2-A): track 0.00 -> 1.95 mm
Other:
- board text added: "IN"
- board text added: "OUT"
- board text added: "XNP 1.1"
